File: src/ESP32-Modular-Board.kicad_sch (KiCad schematic)
At the start: 59 parts, among them J1 UART, J2 USB_C_Receptacle_PowerOnly_6P, J3 Conn_01x06_Socket, SW1 BOOT, SW2 RESET, SW3 SW_Push, SW4 SW_Push, SW5 SW_Push, SW6 SW_Push, SW7 SW_Push, U1 AMS1117-3.3, U2 HT6873B5SPNR, U3 ESP32-MINI-1-N4, U4 MT3608, U5 TP4056-42-ESOP8

Commit message: Added pictures
Other:
- note added: "0"
- note added: "12-06-2025"
- note added: "ReVibe ESP32 Audio PCB Prototype"
Changed lines of the file:
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@@
+		)
+	)
+	(text "0"
+		(exclude_from_sim no)
+		(at 268.986 193.548 0)
+		(effects
+			(font
+				(size 1.778 1.778)
+			)
 		)
 	)
@@
 			)
 		)
+	)
+	(text "12-06-2025"
+		(exclude_from_sim no)
+		(at 215.138 193.294 0)
+		(effects
+			(font
+				(size 1.778 1.778)
+			)
+		)
+	)
+	(text "ReVibe ESP32 Audio PCB Prototype"
+		(exclude_from_sim no)
+		(at 210.058 189.738 0)
+		(effects
+			(font
+				(size 1.778 1.778)
+			)
+		)
